Commit message: Add files via upload

File: ixnaminki_olinki_ws/src/ixnaminki2_description/urdf/brazo.urdf.xacro (robot description, xacro)
@@ -225,5 +225,5 @@
         <origin xyz="0.0 0.0 ${esc*74}" rpy="0.0 0.0 0.3"/>
         <axis xyz="0 1 0"/>
-        <limit lower="-1.7" upper="1.3" effort="1.0" velocity="5.0"/>
+        <limit lower="-2.077" upper="1.11" effort="1.0" velocity="5.0"/>
     </joint>
     <joint name="joint_upper" type="revolute">
@@ -232,5 +232,5 @@
         <origin xyz="${esc*255.14} 0.0 ${esc*405.5}" rpy="0.0 0.0 0.0"/>
         <axis xyz="0 1 0"/>
-        <limit lower="-2.0" upper="1.2" effort="1.0" velocity="5.0"/>
+        <limit lower="-1.66" upper="1.39" effort="1.0" velocity="5.0"/>
     </joint>
     <joint name="joint_rotative" type="revolute">

Commit message: Add files via upload

File: ixnaminki_olinki_ws/src/ixnaminki2_description/urdf/brazo.urdf.xacro (robot description, xacro)
@@ -244,7 +244,8 @@
         <parent link="rotative_arm"/>
         <child link="wrist"/>
-        <origin xyz="${esc*176} 0 0" rpy="0 0 0"/>
+        <origin xyz="${esc*176} 0 0" rpy="0 -0.6 0"/>
         <axis xyz="0 1 0"/>
-        <limit lower="-2.5" upper="1.0" effort="1.0" velocity="5.0"/>
+        <!--limit lower="-2.5" upper="1.0" effort="1.0" velocity="5.0"/-->
+        <limit lower="-0.005" upper="0.005" effort="1.0" velocity="5.0"/>
     </joint>
     <joint name="joint_wrist_gripper" type="fixed">
